File: eduardo-contador/PCB_Contador/PCB_Contador.kicad_pcb (KiCad board)
At the start: 2 copper layers, 57 parts, among them J1 Screw_Terminal_01x02, SW1 SW_DIP_x04, SW3 SW_DIP_x04, SW4 SW_DIP_x04, U1 74LS47, U2 74LS190, U3 74LS47, U4 74LS190, U5 74LS190, U6 74LS47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

Commit message: cambios eduardo
Actualizacion
Routing:
- net GND: track 379.4 -> 169.9 mm, vias 18 -> 5
- net PAUSA: track 166.1 -> 163.0 mm
- net Net-(U2-Rc): track 48.8 -> 46.2 mm
- net Net-(U3-c): track 21.7 -> 19.5 mm
- net Net-(U3-b): track 36.7 -> 34.6 mm
- net Net-(U3-f): track 121.9 -> 120.1 mm
- net Net-(U1-c): track 23.0 -> 21.4 mm
- net Net-(U2-Q2): track 16.1 -> 14.5 mm
- net Net-(U3-e): track 27.5 -> 26.2 mm
- net Net-(U5-P0): track 47.1 -> 45.8 mm
- net Net-(U1-C): track 15.9 -> 14.7 mm
- net Net-(U4-P0): track 47.4 -> 46.1 mm
- net Vcc: track 851.0 -> 850.1 mm
- net Net-(U1-b): track 39.0 -> 38.2 mm
- net Net-(U3-g): track 94.8 -> 94.2 mm
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
Commit message: CASI FINAL
Routing:
- net Vcc: track 850.1 -> 845.7 mm
- net Net-(U1-g): track 87.9 -> 85.5 mm
- net Net-(U1-f): track 105.0 -> 104.4 mm
Other:
- board outline added: 134.6 x 124.5 mm
