File: ivan-joel/Amplificador_D/Amplificador_D.kicad_pcb (KiCad board)
At the start: 2 copper layers, 59 parts, among them J1 Conn_01x02, J2 Conn_01x02, J3 Conn_01x02, J4 Conn_01x02, Q1 IRFZ44N, Q2 IRFZ44N, SW1 SW_SPDT_321, U1 L78L09_TO92, U2 LM358, U3 TL494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

Commit message: cambiso antes del merge
Parts:
- moved C9 275.0 mm to (72.3, 104.1)
- moved R8 271.9 mm to (70.9, 74.0)
- moved R9 271.9 mm to (70.9, 77.1)
- moved U4 209.8 mm to (100.1, 80.5)
- moved R7 195.8 mm to (70.9, 70.8)
- moved C12 193.5 mm to (90.4, 113.4)
- moved C13 193.5 mm to (90.2, 56.1)
- moved C15 193.5 mm to (90.2, 79.2)
- moved C16 193.5 mm to (110.9, 112.3)
- moved C17 193.5 mm to (123.7, 74.8)
- moved D1 193.5 mm to (116.8, 108.0)
- moved D2 193.5 mm to (116.8, 112.2)
- moved D3 193.5 mm to (116.8, 116.5)
- moved L1 193.5 mm to (102.0, 57.4)
- moved L2 193.5 mm to (102.0, 71.4)
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Routing:
- net GND: track 83.2 -> 0.00 mm
- net +12V: track 19.3 -> 0.00 mm
- net Net-(J2-Pin_1): track 18.9 -> 0.00 mm
- net VDC: track 11.0 -> 0.00 mm
- net Net-(C1-Pad2): track 5.19 -> 0.00 mm
- net Net-(U1-VO): track 3.72 -> 0.00 mm
- added copper zone on F.Cu, net GND
Other:
- board outline added: 79.5 x 76.5 mm
