File: aldo-antonella-555/Tier 555/Tier 555.kicad_sch (KiCad schematic)
At the start: 51 parts, among them J1 GND, J2 Trigger, J3 Output, J4 Reset, J5 Control Voltage, J6 Threshold, J7 Discharge, J8 Vcc, Q1 2N3904, Q10 2N3906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

Commit message: parte del timer 555
Parts:
- J1, J2, J3, J4, J5, J6, J7, J8: footprint (none) -> Connector_PinHeader_2.54mm:PinHeader_1x01_P2.54mm_Vertical
- R1, R10, R11, R12, R13, R14, R15, R16, R17, R2, R3, R4, R5, R6, R7, R8, R9: footprint (none) -> Resistor_THT:R_Axial_DIN0207_L6.3mm_D2.5mm_P10.16mm_Horizontal
Connections:
- net Earth renamed GND
