File: aldo-antonella-555/N555/KICAD/CONFIGURACIÓN MONOSTABLE K/CONFIGURACIÓN MONOSTABLE K.kicad_sch (KiCad schematic)
At the start: 9 parts, among them J1 Conn_01x02_Socket, SW1 SW_SPST, U1 LM555xM

Commit message: CASI FINAL
Parts:
- removed SW1: SW_SPST, symbol Switch:SW_SPST
- added C3, C4: C, symbol Device:C
- added D2: LED, symbol Device:LED
- added J2: Conn_01x04_Pin, Connector_PinHeader_2.54mm:PinHeader_1x04_P2.54mm_Vertical, symbol Connector:Conn_01x04_Pin
- added R3, R4: R, symbol Device:R
- added RV2: R_Potentiometer, symbol Device:R_Potentiometer
- added S1: TL59NF160Q, TL59NF160Q:SW_TL59NF160Q, symbol TL59NF160Q:TL59NF160Q
- added U2: LM555xM, Package_SO:SOIC-8_3.9x4.9mm_P1.27mm, symbol Timer:LM555xM
Connections:
- net VCC: now reaches C1.1, J1.2 (Pin_2), R1.1, R1.2, RV1.3, U1.2 (TR), U1.4 (R), U1.5 (CV), U1.8 (VCC)
- net VCC: now also R3.1, S1.2, U2.8 (VCC)
- net GND: now reaches C1.2, C2.2, D1.1 (K), J1.1 (Pin_1), U1.1 (GND)
- net GND: now also C3.2, C4.2, D2.1 (K), S1.1, U2.1 (GND)
- net at RV1.1: now also C2.1, RV1.2, U1.6 (THR), U1.7 (DIS)
- net MONO: now reaches U1.3 (Q)
- net MONO: now also J2.1 (Pin_1); no longer R2.1
- new net: C4.1, RV2.1, RV2.2, U2.2 (TR), U2.6 (THR)
- new net: R3.2, RV2.3, U2.7 (DIS)
- new net: C3.1, U2.5 (CV)
- new net: D2.2 (A), R4.1
- new net AST: J2.3 (Pin_3), U2.3 (Q)
- new net ASTL: J2.4 (Pin_4), R4.2
- new net MONOL: J2.2 (Pin_2), R2.1
- no-connect marks 0 -> 1
Other:
- moved on the sheet: C1, C2, D1, J1, R1, R2, RV1, U1

Commit message: Hola cambios final
Parts:
- C1, C2, C3, C4: footprint (none) -> Capacitor_THT:CP_Radial_Tantal_D4.5mm_P5.00mm
- D1, D2: footprint (none) -> LED_THT:LED_D8.0mm
- J1: footprint (none) -> Connector_PinHeader_2.54mm:PinHeader_1x02_P2.54mm_Vertical
- R1, R2, R3, R4: footprint (none) -> Resistor_THT:R_Axial_DIN0207_L6.3mm_D2.5mm_P10.16mm_Horizontal
- RV1, RV2: footprint (none) -> Potentiometer_THT:Potentiometer_Omeg_PC16BU_Vertical
- U1, U2: footprint Package_SO:SOIC-8_3.9x4.9mm_P1.27mm -> Package_DIP:DIP-8_W7.62mm_LongPads
Connections:
- net MONO: now also J2.2 (Pin_2); no longer J2.1 (Pin_1)
- net MONOL: now also J2.1 (Pin_1); no longer J2.2 (Pin_2)
- net VCC: now also U2.4 (R); no longer C1.1, R1.2, S1.2, U1.2 (TR), U1.5 (CV)
- new net: R1.2, S1.2, U1.2 (TR)
- new net: C1.1, U1.5 (CV)
- no-connect marks 1 -> 0
Changed lines of the file:
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@@
+	)
+	(junction
+		(at 123.19 46.99)
+		(diameter 0)
+		(color 0 0 0 0)
 	)
 	(junction
@@
 	)
 	(junction
-		(at 124.46 46.99)
-		(diameter 0)
-		(color 0 0 0 0)
-	)
-	(junction
-		(at 124.46 52.07)
+		(at 123.19 39.37)
 		(diameter 0)
 		(color 0 0 0 0)
@@
 	)
 	(junction
-		(at 124.46 57.15)
-		(diameter 0)
-		(color 0 0 0 0)
-	)
-	(junction
 		(at 161.29 130.81)
-		(diameter 0)
-		(color 0 0 0 0)
-	)
-	(junction
-		(at 124.46 39.37)
 		(diameter 0)
 		(color 0 0 0 0)
@@
 		(color 0 0 0 0)
 	)
-	(no_connect
-		(at 123.19 123.19)
-	)
-	(wire
-		(pts
-			(xy 124.46 46.99) (xy 124.46 39.37)
+	(wire
+		(pts
+			(xy 123.19 46.99) (xy 123.19 39.37)
 		)
 		(stroke
@@
 	(wire
 		(pts
-			(xy 124.46 39.37) (xy 124.46 38.1)
+			(xy 123.19 39.37) (xy 123.19 38.1)
 		)
 		(stroke
@@
 	(wire
 		(pts
+			(xy 120.65 123.19) (xy 120.65 106.68)
+		)
+		(stroke
+			(width 0)
+			(type default)
+		)
+	)
+	(wire
+		(pts
 			(xy 124.46 57.15) (xy 120.65 57.15)
 		)
@@
 	(wire
 		(pts
-			(xy 124.46 52.07) (xy 124.46 46.99)
+			(xy 123.19 46.99) (xy 123.19 62.23)
 		)
 		(stroke
@@
 	(wire
 		(pts
-			(xy 113.03 39.37) (xy 124.46 39.37)
+			(xy 113.03 39.37) (xy 123.19 39.37)
 		)
 		(stroke
@@
 	(wire
 		(pts
-			(xy 124.46 57.15) (xy 124.46 52.07)
-		)
-		(stroke
-			(width 0)
-			(type default)
-		)
-	)
-	(wire
-		(pts
 			(xy 73.66 43.18) (xy 73.66 48.26)
 		)
@@
 	(wire
 		(pts
+			(xy 123.19 62.23) (xy 124.46 62.23)
+		)
+		(stroke
+			(width 0)
+			(type default)
+		)
+	)
+	(wire
+		(pts
 			(xy 120.65 57.15) (xy 120.65 64.77)
 		)
@@
 	(wire
 		(pts
+			(xy 123.19 39.37) (xy 166.37 39.37)
+		)
+		(stroke
+			(width 0)
+			(type default)
+		)
+	)
+	(wire
+		(pts
 			(xy 156.21 76.2) (xy 156.21 81.28)
 		)
@@
 	(wire
 		(pts
-			(xy 124.46 39.37) (xy 166.37 39.37)
-		)
-		(stroke
-			(width 0)
-			(type default)
-		)
-	)
-	(wire
-		(pts
 			(xy 161.29 49.53) (xy 161.29 54.61)
 		)
@@
 	(wire
 		(pts
-			(xy 124.46 62.23) (xy 124.46 57.15)
-		)
-		(stroke
-			(width 0)
-			(type default)
-		)
-	)
-	(wire
-		(pts
 			(xy 113.03 52.07) (xy 113.03 60.96)
 		)
@@
 	(wire
 		(pts
+			(xy 120.65 106.68) (xy 135.89 106.68)
+		)
+		(stroke
+			(width 0)
+			(type default)
+		)
+	)
+	(wire
+		(pts
 			(xy 161.29 54.61) (xy 166.37 54.61)
 		)
@@
 	(wire
 		(pts
+			(xy 123.19 46.99) (xy 137.16 46.99)
+		)
+		(stroke
+			(width 0)
+			(type default)
+		)
+	)
+	(wire
+		(pts
 			(xy 166.37 53.34) (xy 166.37 54.61)
 		)
@@
 	(wire
 		(pts
-			(xy 124.46 46.99) (xy 137.16 46.99)
-		)
-		(stroke
-			(width 0)
-			(type default)
-		)
-	)
-	(wire
-		(pts
 			(xy 151.13 52.07) (xy 151.13 49.53)
 		)
@@
 		)
 	)
-	(global_label "MONO"
+	(wire
+		(pts
+			(xy 123.19 123.19) (xy 120.65 123.19)
+		)
+		(stroke
+			(width 0)
+			(type default)
+		)
+	)
+	(global_label "MONOL"
 		(shape input)
 		(at 189.23 78.74 0)
@@
 		)
 		(property "Intersheetrefs" "${INTERSHEET_REFS}"
-			(at 197.6581 78.74 0)
+			(at 198.6862 78.74 0)
 			(effects
 				(font
@@
 		)
 	)
-	(global_label "MONOL"
+	(global_label "MONO"
 		(shape input)
 		(at 189.23 81.28 0)
@@
 		)
 		(property "Intersheetrefs" "${INTERSHEET_REFS}"
-			(at 198.6862 81.28 0)
+			(at 197.6581 81.28 0)
 			(effects
 				(font
@@
 			)
 		)
-		(property "Footprint" ""
+		(property "Footprint" "Resistor_THT:R_Axial_DIN0207_L6.3mm_D2.5mm_P10.16mm_Horizontal"
 			(at 111.252 45.72 90)
 			(effects
@@
 			)
 		)
-		(property "Footprint" ""
+		(property "Footprint" "Potentiometer_THT:Potentiometer_Omeg_PC16BU_Vertical"
 			(at 161.29 125.73 0)
 			(effects
@@
 			)
 		)
-		(property "Footprint" ""
+		(property "Footprint" "Capacitor_THT:CP_Radial_Tantal_D4.5mm_P5.00mm"
 			(at 120.3452 139.7 0)
 			(effects
@@
 			)
 		)
-		(property "Footprint" ""
+		(property "Footprint" "Resistor_THT:R_Axial_DIN0207_L6.3mm_D2.5mm_P10.16mm_Horizontal"
 			(at 159.512 111.76 90)
 			(effects
@@
 			)
 		)
-		(property "Footprint" ""
+		(property "Footprint" "Connector_PinHeader_2.54mm:PinHeader_1x02_P2.54mm_Vertical"
 			(at 68.58 50.8 0)
 			(effects
@@
 			)
 		)
-		(property "Footprint" ""
+		(property "Footprint" "Potentiometer_THT:Potentiometer_Omeg_PC16BU_Vertical"
 			(at 166.37 49.53 0)
 			(effects
@@
 	(symbol
 		(lib_id "power:VCC")
-		(at 124.46 38.1 0)
+		(at 123.19 38.1 0)
 		(unit 1)
 		(exclude_from_sim no)
@@
 		(fields_autoplaced yes)
 		(property "Reference" "#PWR02"
-			(at 124.46 41.91 0)
+			(at 123.19 41.91 0)
 			(effects
 				(font
@@
 		)
 		(property "Value" "VCC"
-			(at 124.46 33.02 0)
+			(at 123.19 33.02 0)
 			(effects
 				(font
@@
 		)
 		(property "Footprint" ""
-			(at 124.46 38.1 0)
+			(at 123.19 38.1 0)
 			(effects
 				(font
@@
 		)
 		(property "Datasheet" ""
-			(at 124.46 38.1 0)
+			(at 123.19 38.1 0)
 			(effects
 				(font
@@
 		)
 		(property "Description" "Power symbol creates a global label with name \"VCC\""
-			(at 124.46 38.1 0)
+			(at 123.19 38.1 0)
 			(effects
 				(font
@@
 			)
 		)
-		(property "Footprint" "Package_SO:SOIC-8_3.9x4.9mm_P1.27mm"
+		(property "Footprint" "Package_DIP:DIP-8_W7.62mm_LongPads"
 			(at 158.75 67.31 0)
 			(effects
@@
 			)
 		)
-		(property "Footprint" "Package_SO:SOIC-8_3.9x4.9mm_P1.27mm"
+		(property "Footprint" "Package_DIP:DIP-8_W7.62mm_LongPads"
 			(at 157.48 128.27 0)
 			(effects
@@
 			)
 		)
-		(property "Footprint" ""
+		(property "Footprint" "LED_THT:LED_D8.0mm"
 			(at 171.45 127 0)
 			(effects
@@
 			)
 		)
-		(property "Footprint" ""
+		(property "Footprint" "Capacitor_THT:CP_Radial_Tantal_D4.5mm_P5.00mm"
 			(at 121.6152 72.39 0)
 			(effects
@@
 			)
 		)
-		(property "Footprint" ""
+		(property "Footprint" "Resistor_THT:R_Axial_DIN0207_L6.3mm_D2.5mm_P10.16mm_Horizontal"
 			(at 154.432 62.23 90)
 			(effects
@@
 			)
 		)
-		(property "Footprint" ""
+		(property "Footprint" "LED_THT:LED_D8.0mm"
 			(at 156.21 72.39 0)
 			(effects
@@
 			)
 		)
-		(property "Footprint" ""
+		(property "Footprint" "Capacitor_THT:CP_Radial_Tantal_D4.5mm_P5.00mm"
 			(at 167.3352 73.66 0)
 			(effects
@@
 			)
 		)
-		(property "Footprint" ""
+		(property "Footprint" "Capacitor_THT:CP_Radial_Tantal_D4.5mm_P5.00mm"
 			(at 162.2552 139.7 0)
 			(effects
@@
 			)
 		)
-		(property "Footprint" ""
+		(property "Footprint" "Resistor_THT:R_Axial_DIN0207_L6.3mm_D2.5mm_P10.16mm_Horizontal"
 			(at 173.228 111.76 90)
 			(effects
