File: helton-tl494/TL494/TL494/TL494NUEVA-VERSION.kicad_pcb (KiCad board)
At the start: 2 copper layers, 39 parts, among them J1 Jumper E1, J2 Jumper E1, J3 +-, J4 Vout1, J5 Vout1, J6 Conn_02x02_Odd_Even, J7 Vout1, J8 Conn_02x04_Odd_Even, Q1 NMOS, Q2 NMOS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

Commit message: CASI FINAL
Parts:
- moved C1 1.57 mm to (153.4, 69.1)
- moved R1 1.49 mm to (156.5, 69.2)
- moved R12 1.22 mm to (159.8, 79.3)
Routing:
- net GNDREF: track 304.0 -> 10.7 mm
- net 1IN+: track 26.9 -> 29.1 mm
- net CT: track 5.54 -> 4.26 mm
- net RT: track 4.78 -> 4.16 mm
